Commit message: feat: add moveit2 configuration

File: src/rover_urdf_pkg/urdf/ASTRA_Arm.urdf (robot description, URDF)
Before this commit: robot ASTRA Arm, 9 links, 8 joints
Joints:
- removed joint Axis 0 Joint
- removed joint Axis 1 Joint
- removed joint Axis 2 Joint
- removed joint Axis 3 Joint
- removed joint Gripper Slider Left
- removed joint Gripper Slider Right
- removed joint Wrist Differential Joint
- removed joint Wrist-EF Roll Joint
- added joint Axis_0_Joint: type revolute, parent base_link, child Axis 0 Plate, origin xyz=0.018772 -0.020734 -0.04971 rpy=1.5708 0 3.1115, axis 0 -1 0, limit lower=-3.14 upper=3.14 effort=0 velocity=0.05
- added joint Axis_1_Joint: type revolute, parent Axis 0 Plate, child Axis 1 Segment, origin xyz=-0.0271654135185528 0.0927245490180083 0.00384109909109076 rpy=-3.14159265358977 -0.00524713054608625 1.5707963267949, axis 0 -1 0, limit lower=-1.05 upper=1.6 effort=0 velocity=0.05
- added joint Axis_2_Joint: type revolute, parent Axis 1 Segment, child Axis 2 Segment, origin xyz=0.470027000000004 0.0126999999999999 0 rpy=3.14159265358979 0.000449358059257729 0, axis 0 -1 0, limit lower=-2.0 upper=2.0 effort=0 velocity=0.05
- added joint Axis_3_Joint: type revolute, parent Axis 2 Segment, child Wrist, origin xyz=0.393826999999998 0 0 rpy=0 -0.000409495780687665 0, axis 0 -1 0, limit lower=-1.6 upper=1.9 effort=0 velocity=0.05
- added joint Gripper _Slider_Right: type prismatic, parent End Effector, child EF Gripper Right, origin xyz=0 0 -0.031677 rpy=0 0 3.1416, axis 0 1 0, limit lower=-0.025 upper=0.04 effort=0 velocity=0.05
- added joint Gripper_Slider_Left: type prismatic, parent End Effector, child EF Gripper Left, origin xyz=0 0 -0.031677 rpy=0 0 0, axis 0 -1 0, limit lower=-0.04 upper=0.025 effort=0 velocity=0.05
- added joint Wrist-EF_Roll_Joint: type continuous, parent Diff Carrier, child End Effector, origin xyz=0 0.01 0 rpy=-1.5708 -0.21566 -3.1416, axis 0 0 1
- added joint Wrist_Differential_Joint: type revolute, parent Wrist, child Diff Carrier, origin xyz=0.176692001200001 -0.00622300000004081 0 rpy=-3.05263944120951 1.57079631189374 1.65994236547327, axis -1 0 0, limit lower=-1.6 upper=1.6 effort=0 velocity=0.05

Commit message: fix: move roll joint to arm pose group, add real velocity limit to grippers

File: src/rover_urdf_pkg/urdf/ASTRA_Arm.urdf (robot description, URDF)
Before this commit: robot ASTRA_Arm, 9 links, 8 joints
Joints:
- joint Gripper_Slider_Left: limit lower=-0.04 upper=0.025 effort=0 velocity=3.1415963 -> lower=-0.04 upper=0.025 effort=0 velocity=0.015
- joint Gripper_Slider_Right: limit lower=-0.025 upper=0.04 effort=0 velocity=3.1415963 -> lower=-0.025 upper=0.04 effort=0 velocity=0.015; mimic (none) -> joint=Gripper_Slider_Left multiplier=-1
