Commit message: refactor: re-ran setup assistant

File: src/astra_arm_moveit_config/config/ASTRA_Arm.ros2_control.xacro (robot description, xacro)
@@ -56,4 +56,12 @@
                 <state_interface name="velocity"/>
             </joint>
+            <joint name="Gripper _Slider_Right">
+                <command_interface name="position"/>
+                <command_interface name="velocity"/>
+                <state_interface name="position">
+                  <param name="initial_value">${initial_positions['Gripper _Slider_Right']}</param>
+                </state_interface>
+                <state_interface name="velocity"/>
+            </joint>
             <joint name="Gripper_Slider_Left">
                 <command_interface name="position"/>
@@ -64,12 +72,4 @@
                 <state_interface name="velocity"/>
             </joint>
-            <joint name="Gripper _Slider_Right">
-                <command_interface name="position"/>
-                <command_interface name="velocity"/>
-                <state_interface name="position">
-                  <param name="initial_value">${initial_positions['Gripper _Slider_Right']}</param>
-                </state_interface>
-                <state_interface name="velocity"/>
-            </joint>
         </ros2_control>
     </xacro:macro>

Commit message: fix: remove space from joint name

File: src/astra_arm_moveit_config/config/ASTRA_Arm.ros2_control.xacro (robot description, xacro)
@@ -56,9 +56,9 @@
                 <state_interface name="velocity"/>
             </joint>
-            <joint name="Gripper _Slider_Right">
+            <joint name="Gripper_Slider_Right">
                 <command_interface name="position"/>
                 <command_interface name="velocity"/>
                 <state_interface name="position">
-                  <param name="initial_value">${initial_positions['Gripper _Slider_Right']}</param>
+                  <param name="initial_value">${initial_positions['Gripper_Slider_Right']}</param>
                 </state_interface>
                 <state_interface name="velocity"/>

File: src/rover_urdf_pkg/urdf/ASTRA_Arm.urdf (robot description, URDF)
Before this commit: robot ASTRA_Arm, 9 links, 8 joints
Joints:
- removed joint Gripper _Slider_Right
- added joint Gripper_Slider_Right: type prismatic, parent End Effector, child EF Gripper Right, origin xyz=0 0 -0.031677 rpy=0 0 3.1416, axis 0 1 0, limit lower=-0.025 upper=0.04 effort=0 velocity=3.1415963
- joint Axis_0_Joint: limit lower=-3.14 upper=3.14 effort=0 velocity=0.05 -> lower=-3.14 upper=3.14 effort=0 velocity=3.1415963
- joint Axis_1_Joint: limit lower=-1.05 upper=1.6 effort=0 velocity=0.05 -> lower=-1.05 upper=1.6 effort=0 velocity=3.1415963
- joint Axis_2_Joint: limit lower=-2.0 upper=2.0 effort=0 velocity=0.05 -> lower=-2.0 upper=2.0 effort=0 velocity=3.1415963
- joint Axis_3_Joint: limit lower=-1.6 upper=1.9 effort=0 velocity=0.05 -> lower=-1.6 upper=1.9 effort=0 velocity=3.1415963
- joint Gripper_Slider_Left: limit lower=-0.04 upper=0.025 effort=0 velocity=0.05 -> lower=-0.04 upper=0.025 effort=0 velocity=3.1415963
- joint Wrist_Differential_Joint: limit lower=-1.6 upper=1.6 effort=0 velocity=0.05 -> lower=-1.6 upper=1.6 effort=0 velocity=3.1415963

Commit message: fix: grippers now act correctly

File: src/astra_arm_moveit_config/config/ASTRA_Arm.ros2_control.xacro (robot description, xacro)
@@ -56,12 +56,4 @@
                 <state_interface name="velocity"/>
             </joint>
-            <joint name="Gripper_Slider_Right">
-                <command_interface name="position"/>
-                <command_interface name="velocity"/>
-                <state_interface name="position">
-                  <param name="initial_value">${initial_positions['Gripper_Slider_Right']}</param>
-                </state_interface>
-                <state_interface name="velocity"/>
-            </joint>
             <joint name="Gripper_Slider_Left">
                 <command_interface name="position"/>
