Commit message: refactor: post-comp IK testing

File: src/arm_pkg/urdf/arm12.urdf (robot description, URDF)
Before this commit: robot robot, 12 links, 11 joints
Joints:
- joint Axis_2_Joint: limit lower=-1.6 upper=1.6 effort=1000.0 velocity=0.5 -> lower=-2.7 upper=2.7 effort=1000.0 velocity=0.5

Commit message: feat: add viz code from Tristan's ik_test and add CAD to URDF

File: src/arm_pkg/urdf/arm12.urdf (robot description, URDF)
Before this commit: robot robot, 12 links, 11 joints
Links:
- removed link Axis_0
- added link Axis_0_Plate, mass 1; collision cylinder length=0.059 radius=0.15; visual mesh filename=package://arm_pkg/urdf/Axis 0 Plate.STL scale=1 1 1
- link Axis_1: geometry collision cylinder length=0.1 radius=0.082; visual mesh filename=package://arm_pkg/urdf/Axis 1.STL scale=1 1 1
- link Segment_1: geometry collision cylinder length=0.473 radius=0.025; visual mesh filename=package://arm_pkg/urdf/Segment 1.STL scale=1 1 1
- link base_link: geometry collision box size=0.5 0.5 0.01; visual mesh filename=package://arm_pkg/urdf/Arm Base Plate.STL scale=1 1 1
Joints:
- removed joint Axis_0_Joint
- added joint Axis_0: type revolute, parent base_link, child Axis_0_Plate, origin xyz=0 0 0.035 rpy=0 0 0, axis 0 0 1, limit lower=-2.5 upper=2.5 effort=1000.0 velocity=0.5
- joint Axis_1_Joint: parent Axis_0 -> Axis_0_Plate

Commit message: fix: remove spaces from link names to support Jammy
Viz doesn't work when the links have spaces in their names on Jammy ._.

File: src/arm_pkg/urdf/arm12.urdf (robot description, URDF)
Before this commit: robot robot, 12 links, 11 joints
Links:
- link Axis_0_Plate: geometry collision cylinder length=0.059 radius=0.15; visual mesh filename=package://arm_pkg/urdf/Axis_0_Plate.STL scale=1 1 1

File: src/rover_urdf_pkg/urdf/ASTRA_Arm.urdf (robot description, URDF)
Before this commit: robot ASTRA_Arm, 9 links, 8 joints
Links:
- removed link Axis 0 Plate
- removed link Axis 1 Segment
- removed link Axis 2 Segment
- removed link Diff Carrier
- removed link EF Gripper Left
- removed link EF Gripper Right
- removed link End Effector
- added link Axis_0_Plate, mass 2.045; collision mesh filename=package://rover_urdf_pkg/meshes/Axis_0_Plate.STL; visual mesh filename=package://rover_urdf_pkg/meshes/Axis_0_Plate.STL
- added link Axis_1_Segment, mass 2.10107115350287; collision mesh filename=package://rover_urdf_pkg/meshes/Axis_1_Segment.STL; visual mesh filename=package://rover_urdf_pkg/meshes/Axis_1_Segment.STL
- added link Axis_2_Segment, mass 3.13644489009951; collision mesh filename=package://rover_urdf_pkg/meshes/Axis_2_Segment.STL; visual mesh filename=package://rover_urdf_pkg/meshes/Axis_2_Segment.STL
- added link Diff_Carrier, mass 0.0655351660884378; collision mesh filename=package://rover_urdf_pkg/meshes/Diff_Carrier.STL; visual mesh filename=package://rover_urdf_pkg/meshes/Diff_Carrier.STL
- added link EF_Gripper_Left, mass 0.0813132558225319; collision mesh filename=package://rover_urdf_pkg/meshes/EF_Gripper_Left.STL; visual mesh filename=package://rover_urdf_pkg/meshes/EF_Gripper_Left.STL
- added link EF_Gripper_Right, mass 0.0859306256217421; collision mesh filename=package://rover_urdf_pkg/meshes/EF_Gripper_Right.STL; visual mesh filename=package://rover_urdf_pkg/meshes/EF_Gripper_Right.STL
- added link End_Effector, mass 0.397605677640027; collision mesh filename=package://rover_urdf_pkg/meshes/End_Effector.STL; visual mesh filename=package://rover_urdf_pkg/meshes/End_Effector.STL
Joints:
- joint Axis_0_Joint: child Axis 0 Plate -> Axis_0_Plate; limit lower=-3.14 upper=3.14 effort=0 velocity=3.1415963 -> lower=-3.14 upper=3.14 effort=0 velocity=31.41593
- joint Axis_1_Joint: child Axis 1 Segment -> Axis_1_Segment; limit lower=-1.05 upper=1.6 effort=0 velocity=3.1415963 -> lower=-1.05 upper=1.6 effort=0 velocity=31.41593; parent Axis 0 Plate -> Axis_0_Plate
- joint Axis_2_Joint: child Axis 2 Segment -> Axis_2_Segment; limit lower=-2.0 upper=2.0 effort=0 velocity=3.1415963 -> lower=-2.0 upper=2.0 effort=0 velocity=31.41593; parent Axis 1 Segment -> Axis_1_Segment
- joint Axis_3_Joint: limit lower=-1.6 upper=1.9 effort=0 velocity=3.1415963 -> lower=-1.6 upper=1.9 effort=0 velocity=31.41593; parent Axis 2 Segment -> Axis_2_Segment
- joint Gripper_Slider_Left: child EF Gripper Left -> EF_Gripper_Left; parent End Effector -> End_Effector
- joint Gripper_Slider_Right: child EF Gripper Right -> EF_Gripper_Right; parent End Effector -> End_Effector
- joint Wrist-EF_Roll_Joint: child End Effector -> End_Effector; parent Diff Carrier -> Diff_Carrier
- joint Wrist_Differential_Joint: child Diff Carrier -> Diff_Carrier; limit lower=-1.6 upper=1.6 effort=0 velocity=3.1415963 -> lower=-1.6 upper=1.6 effort=0 velocity=31.41593
