Commit message: feat: add ros2_control to Core URDF

File: src/core_rover_description/urdf/core_rover.urdf (robot description, URDF)
Before this commit: robot core_rover_description, 8 links, 7 joints
Joints:
- removed joint averaging_bar_axis
- removed joint br_wheel_axis
- added joint averaging_bar_joint: type revolute, parent base_link, child averaging_bar, origin xyz=0 -0.23362 -0.0508 rpy=0 -0.0060774 -3.1416, axis 0 -1 0, limit lower=-0.38 upper=0.38 effort=0 velocity=0, mimic joint=left_suspension_joint multiplier=-1 offset=0
- added joint br_wheel_joint: type continuous, parent right_suspension_member, child br_wheel, origin xyz=-0.41838 -0.17155 0.12984 rpy=0.52965 -1.5708 0, axis -1 0 0
- joint fr_wheel_joint: axis 1 0 0 -> -1 0 0

Commit message: feat: make frames work properly, rviz is now accurate

File: src/core_rover_description/urdf/core_rover.urdf (robot description, URDF)
Before this commit: robot core_rover_description, 8 links, 7 joints
Links:
- added link dummy_base_link
Joints:
- added joint dummy_base_link_joint: type fixed, parent dummy_base_link, child base_link, origin xyz=0 0 0.35 rpy=0 0 1.5707963267948966, axis 0 0 0

File: src/core_rover_description/urdf/ros2_control.xacro (robot description, xacro)
@@ -5,4 +5,7 @@
             <plugin>gz_ros2_control/GazeboSimSystem</plugin>
         </hardware>
+        <joint name="left_suspension_joint">
+            <state_interface name="position"/>
+        </joint>
         <joint name="bl_wheel_joint">
             <command_interface name="velocity"/>

Commit message: fix: correctly spawn controllers
models was commented out in CMakeLists.txt because it is currently an empty directory, but will be used at a later point

File: src/core_rover_description/urdf/core_rover.urdf (robot description, URDF)
Before this commit: robot core_rover_description, 9 links, 8 joints
Joints:
- joint dummy_base_link_joint: origin xyz=0 0 0.35 rpy=0 0 1.5707963267948966 -> xyz=0 0 0.38 rpy=0 0 1.5707963267948966
