Commit message: style: rename arm urdf packages
* rover_urdf_pkg -> arm_description
* astra_arm_moveit_config -> arm_moveit_config

File: src/arm_description/urdf/ASTRA_Arm.urdf (robot description, URDF)
Before this commit: robot ASTRA_Arm, 9 links, 8 joints
Links:
- link Axis_0_Plate: geometry collision mesh filename=package://arm_description/meshes/Axis_0_Plate.STL; visual mesh filename=package://arm_description/meshes/Axis_0_Plate.STL
- link Axis_1_Segment: geometry collision mesh filename=package://arm_description/meshes/Axis_1_Segment.STL; visual mesh filename=package://arm_description/meshes/Axis_1_Segment.STL
- link Axis_2_Segment: geometry collision mesh filename=package://arm_description/meshes/Axis_2_Segment.STL; visual mesh filename=package://arm_description/meshes/Axis_2_Segment.STL
- link Diff_Carrier: geometry collision mesh filename=package://arm_description/meshes/Diff_Carrier.STL; visual mesh filename=package://arm_description/meshes/Diff_Carrier.STL
- link EF_Gripper_Left: geometry collision mesh filename=package://arm_description/meshes/EF_Gripper_Left.STL; visual mesh filename=package://arm_description/meshes/EF_Gripper_Left.STL
- link EF_Gripper_Right: geometry collision mesh filename=package://arm_description/meshes/EF_Gripper_Right.STL; visual mesh filename=package://arm_description/meshes/EF_Gripper_Right.STL
- link End_Effector: geometry collision mesh filename=package://arm_description/meshes/End_Effector.STL; visual mesh filename=package://arm_description/meshes/End_Effector.STL
- link Wrist: geometry collision mesh filename=package://arm_description/meshes/Wrist.STL; visual mesh filename=package://arm_description/meshes/Wrist.STL
- link base_link: geometry collision mesh filename=package://arm_description/meshes/base_link.STL; visual mesh filename=package://arm_description/meshes/base_link.STL

File: src/arm_moveit_config/config/ASTRA_Arm.urdf.xacro (robot description, xacro)
@@ -3,5 +3,5 @@
     <xacro:arg name="initial_positions_file" default="initial_positions.yaml" />
     <!-- Import ASTRA_Arm urdf file -->
-    <xacro:include filename="$(find rover_urdf_pkg)/urdf/ASTRA_Arm.urdf" />
+    <xacro:include filename="$(find arm_description)/urdf/ASTRA_Arm.urdf" />
     <!-- Import control_xacro -->
     <xacro:include filename="ASTRA_Arm.ros2_control.xacro" />
