Commit message: style: rename core_rover_description to core_description

File: src/astra_description/core_description/urdf/core_rover.urdf (robot description, URDF)
Before this commit: robot core_rover_description, 9 links, 8 joints
Links:
- link averaging_bar: geometry collision mesh filename=package://core_description/meshes/averaging_bar.STL; visual mesh filename=package://core_description/meshes/averaging_bar.STL
- link base_link: geometry collision mesh filename=package://core_description/meshes/base_link.STL; visual mesh filename=package://core_description/meshes/base_link.STL
- link bl_wheel: geometry collision mesh filename=package://core_description/meshes/bl_wheel.STL; visual mesh filename=package://core_description/meshes/bl_wheel.STL
- link br_wheel: geometry collision mesh filename=package://core_description/meshes/br_wheel.STL; visual mesh filename=package://core_description/meshes/br_wheel.STL
- link fl_wheel: geometry collision mesh filename=package://core_description/meshes/fl_wheel.STL; visual mesh filename=package://core_description/meshes/fl_wheel.STL
- link fr_wheel: geometry collision mesh filename=package://core_description/meshes/fr_wheel.STL; visual mesh filename=package://core_description/meshes/fr_wheel.STL
- link left_suspension_member: geometry collision mesh filename=package://core_description/meshes/left_suspension_member.STL; visual mesh filename=package://core_description/meshes/left_suspension_member.STL
- link right_suspension_member: geometry collision mesh filename=package://core_description/meshes/right_suspension_member.S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; visual mesh filename=package://core_description/meshes/right_suspension_member.S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

File: src/astra_description/core_description/urdf/ros2_control.xacro (robot description, xacro)
@@ -31,5 +31,5 @@
     <gazebo>
         <plugin filename="gz_ros2_control-system" name="gz_ros2_control::GazeboSimROS2ControlPlugin">
-            <parameters>$(find core_rover_description)/config/ros2_controllers.yaml</parameters>
+            <parameters>$(find core_description)/config/ros2_controllers.yaml</parameters>
             <ros>
                 <remapping>/diff_controller/cmd_vel_unstamped:=/core/twist</remapping>
